Commit message: change tf publlish

File: config/robot.urdf.xacro (robot description, xacro)
@@ -9,5 +9,13 @@
     <origin xyz="0 0 0" rpy="0 0 0" />
   </joint>
-  <link name="lidar_link"> </link>
+ <!--
+  <link name="os_lidar"> </link>
+  <joint name="lidar_joint" type="fixed">
+    <parent link="base_link" />
+    <child link="os_lidar" />
+    <origin xyz="0 0 0" rpy="0 0 0" />
+  </joint>
+-->
+ <link name="lidar_link"> </link>
   <joint name="lidar_joint" type="fixed">
     <parent link="base_link" />
